Commit message: Update quadruped.urdf

File: src/quadruped/URDF__updated_files/quadruped.urdf (robot description, URDF)
Before this commit: robot quadruped, 13 links, 12 joints
Joints:
- removed joint Right_back_femur_joint
- removed joint Right_back_tibia_joint
- removed joint Right_front_femur_joint
- removed joint Right_front_tibia_joint
- added joint right_back_femur_joint: type revolute, parent Right_back_shoulder, child Right_back_femur, origin xyz=0.0 0.0 0.0 rpy=0 0 0, axis 1 0 0, limit lower=-0.78 upper=0.78 effort=0.1 velocity=0.1
- added joint right_back_tibia_joint: type revolute, parent Right_back_femur, child Right_back_tibia, origin xyz=0.0 0.0 0.0 rpy=0 0 0, axis 1 0 0, limit lower=-0.78 upper=0.78 effort=0.1 velocity=0.1
- added joint right_front_femur_joint: type revolute, parent Right_front_shoulder, child Right_front_femur, origin xyz=0.0 0.0 0.0 rpy=0 0 0, axis 1 0 0, limit lower=-0.78 upper=0.78 effort=0.1 velocity=0.1
- added joint right_front_tibia_joint: type revolute, parent Right_front_femur, child Right_front_tibia, origin xyz=0.0 0.0 0.0 rpy=0 0 0, axis 1 0 0, limit lower=-0.78 upper=0.78 effort=0.1 velocity=0.1

Commit message: Add files via upload

File: src/quadruped/URDF__updated_files/quadruped.urdf (robot description, URDF)
Before this commit: robot quadruped, 13 links, 12 joints
Joints:
- joint left_back_femur_joint: origin xyz=0.0 0.0 0.0 rpy=0 0 0 -> xyz=0.0 0.0625 0.0 rpy=0 0 0
- joint left_back_hip_joint: origin xyz=0.0 0.0 0.35 rpy=0 0 0 -> xyz=0.0525 0.1125 0.35 rpy=0 0 0
- joint left_back_tibia_joint: origin xyz=0.0 0.0 0.0 rpy=0 0 0 -> xyz=0.0925 0.092 -0.160 rpy=0 0 0
- joint left_front_femur_joint: origin xyz=0.0 0.0 0.0 rpy=0 0 0 -> xyz=0.0 -0.0625 0.0 rpy=0 0 0
- joint left_front_hip_joint: origin xyz=0.0 0.0 0.35 rpy=0 0 0 -> xyz=0.0525 -0.1125 0.35 rpy=0 0 0
- joint left_front_tibia_joint: origin xyz=0.0 0.0 0.0 rpy=0 0 0 -> xyz=0.0925 0.092 -0.160 rpy=0 0 0
- joint right_back_femur_joint: origin xyz=0.0 0.0 0.0 rpy=0 0 0 -> xyz=0 0.0625 0 rpy=0 0 0
- joint right_back_hip_joint: origin xyz=0 0 0.35 rpy=0 0 0 -> xyz=-0.0525 0.1125 0.35 rpy=0 0 0
- joint right_back_tibia_joint: origin xyz=0.0 0.0 0.0 rpy=0 0 0 -> xyz=-0.0925 0.092 -0.160 rpy=0 0 0
- joint right_front_femur_joint: origin xyz=0.0 0.0 0.0 rpy=0 0 0 -> xyz=0.0 -0.0625 0.0 rpy=0 0 0
- joint right_front_hip_joint: origin xyz=0 0 0.35 rpy=0 0 0 -> xyz=-0.0525 -0.1125 0.35 rpy=0 0 0
- joint right_front_tibia_joint: origin xyz=0.0 0.0 0.0 rpy=0 0 0 -> xyz=-0.0925 0.092 -0.160 rpy=0 0 0
