Commit message: Fixed urdf path

File: src/quadruped/quadruped/pybullet_data/vrka.urdf (robot description, URDF)
Before this commit: robot quadruped, 5 links, 4 joints
Links:
- link base_link: geometry collision mesh filename=package://urdf/base_link_rsz.stl; visual mesh filename=package://urdf/base_link_rsz.stl
- link leftback: geometry collision mesh filename=package://urdf/leftbackleg_rsz.stl; visual mesh filename=package://urdf/leftbackleg_rsz.stl
- link leftfront: geometry collision mesh filename=package://urdf/leftfrontleg_rsz.stl; visual mesh filename=package:///urdf/leftfrontleg_rsz.stl
- link rightback: geometry collision mesh filename=package://urdf/rightbackleg_rsz.stl; visual mesh filename=package://urdf/rightbackleg_rsz.stl
- link rightfront: geometry collision mesh filename=package://urdf/rightfrontleg_rsz.stl; visual mesh filename=package://urdf/rightfrontleg_rsz.stl

Commit message: Update vrka.urdf

File: src/quadruped/quadruped/pybullet_data/vrka.urdf (robot description, URDF)
Before this commit: robot quadruped, 5 links, 4 joints
Joints:
- removed joint leftback_joint
- removed joint leftfront_joint
- removed joint rightback_joint
- removed joint rightfront_joint
- added joint motor_back_left_upper_leg: type revolute, parent base_link, child leftback, origin xyz=0.1 0.273 0.35 rpy=0 0 0, axis 1 0 0, limit lower=-0.78 upper=0.78 effort=0.1 velocity=0.1
- added joint motor_back_right_upper_leg: type revolute, parent base_link, child rightback, origin xyz=-0.1 0.273 0.35 rpy=0 0 0, axis 1 0 0, limit lower=-0.78 upper=0.78 effort=0.1 velocity=0.1
- added joint motor_front_left_upper_leg: type revolute, parent base_link, child leftfront, origin xyz=0.1 -0.075 0.35 rpy=0 0 0, axis 1 0 0, limit lower=-0.7848 upper=0.78 effort=0.1 velocity=0.1
- added joint motor_front_right_upper_leg: type revolute, parent base_link, child rightfront, origin xyz=-0.1 -0.075 0.35 rpy=0 0 0, axis 1 0 0, limit lower=-0.78 upper=0.78 effort=0.1 velocity=0.1

Commit message: Updated kinematics

File: src/quadruped/quadruped/pybullet_data/vrka.urdf (robot description, URDF)
Before this commit: robot quadruped, 5 links, 4 joints
Links:
- removed link leftback
- removed link leftfront
- removed link rightback
- removed link rightfront
- added link Left_back_femur, mass 0.1; collision mesh filename=package://quadruped/meshes/LeftBackFemur.stl scale=0.001 0.001 0.001; visual mesh filename=package://quadruped/meshes/LeftBackFemur.stl scale=0.001 0.001 0.001
- added link Left_back_shoulder, mass 0.1; collision mesh filename=package://quadruped/meshes/LeftBackShoulder.stl scale=0.001 0.001 0.001; visual mesh filename=package://quadruped/meshes/LeftBackShoulder.stl scale=0.001 0.001 0.001
- added link Left_back_tibia, mass 0.1; collision mesh filename=package://quadruped/meshes/LeftBackTibia.stl scale=0.001 0.001 0.001; visual mesh filename=package://quadruped/meshes/LeftBackTibia.stl scale=0.001 0.001 0.001
- added link Left_front_femur, mass 0.1; collision mesh filename=package://quadruped/meshes/LeftFrontFemur.stl scale=0.001 0.001 0.001; visual mesh filename=package://quadruped/meshes/LeftFrontFemur.stl scale=0.001 0.001 0.001
- added link Left_front_shoulder, mass 0.1; collision mesh filename=package://quadruped/meshes/LeftFrontShoulder.stl scale=0.001 0.001 0.001; visual mesh filename=package://quadruped/meshes/LeftFrontShoulder.stl scale=0.001 0.001 0.001
- added link Left_front_tibia, mass 0.1; collision mesh filename=package://quadruped/meshes/LeftFrontTibia.stl scale=0.001 0.001 0.001; visual mesh filename=package://quadruped/meshes/LeftFrontTibia.stl scale=0.001 0.001 0.001
- added link Right_back_femur, mass 0.1; collision mesh filename=package://quadruped/meshes/RightBackFemur.stl scale=0.001 0.001 0.001; visual mesh filename=package://quadruped/meshes/RightBackFemur.stl scale=0.001 0.001 0.001
- added link Right_back_shoulder, mass 0.1; collision mesh filename=package://quadruped/meshes/RightBackShoulder.stl scale=0.001 0.001 0.001; visual mesh filename=package://quadruped/meshes/RightBackShoulder.stl scale=0.001 0.001 0.001
- added link Right_back_tibia, mass 0.1; collision mesh filename=package://quadruped/meshes/RightBackTibia.stl scale=0.001 0.001 0.001; visual mesh filename=package://quadruped/meshes/RightBackTibia.stl scale=0.001 0.001 0.001
- added link Right_front_femur, mass 0.1; collision mesh filename=package://quadruped/meshes/RightFrontFemur.stl scale=0.001 0.001 0.001; visual mesh filename=package://quadruped/meshes/RightFrontFemur.stl scale=0.001 0.001 0.001
- added link Right_front_shoulder, mass 0.1; collision mesh filename=package://quadruped/meshes/RightFrontShoulder.stl scale=0.001 0.001 0.001; visual mesh filename=package://quadruped/meshes/RightFrontShoulder.stl scale=0.001 0.001 0.001
- added link Right_front_tibia, mass 0.1; collision mesh filename=package://quadruped/meshes/RightFrontTibia.stl scale=0.001 0.001 0.001; visual mesh filename=package://quadruped/meshes/RightFrontTibia.stl scale=0.001 0.001 0.001
- link base_link: geometry collision mesh filename=package://quadruped/meshes/chassis_w_motors.stl scale=0.001 0.001 0.001; visual mesh filename=package://quadruped/meshes/chassis_w_motors.stl scale=0.001 0.001 0.001
Joints:
- removed joint leftback_joint
- removed joint leftfront_joint
- removed joint rightback_joint
- removed joint rightfront_joint
- added joint left_back_femur_joint: type revolute, parent Left_back_shoulder, child Left_back_femur, origin xyz=0.0 0.0625 0.0 rpy=0 0 0, axis 1 0 0, limit lower=-0.78 upper=0.78 effort=0.1 velocity=0.1
- added joint left_back_hip_joint: type revolute, parent base_link, child Left_back_shoulder, origin xyz=0.0525 0.1125 0.35 rpy=0 0 0, axis 0 1 0, limit lower=-0.78 upper=0.78 effort=0.1 velocity=0.1
- added joint left_back_tibia_joint: type revolute, parent Left_back_femur, child Left_back_tibia, origin xyz=0.0925 0.092 -0.160 rpy=0 0 0, axis 1 0 0, limit lower=-0.78 upper=0.78 effort=0.1 velocity=0.1
- added joint left_front_femur_joint: type revolute, parent Left_front_shoulder, child Left_front_femur, origin xyz=0.0 -0.0625 0.0 rpy=0 0 0, axis 1 0 0, limit lower=-0.78 upper=0.78 effort=0.1 velocity=0.1
- added joint left_front_hip_joint: type revolute, parent base_link, child Left_front_shoulder, origin xyz=0.0525 -0.1125 0.35 rpy=0 0 0, axis 0 1 0, limit lower=-0.7848 upper=0.78 effort=0.1 velocity=0.1
- added joint left_front_tibia_joint: type revolute, parent Left_front_femur, child Left_front_tibia, origin xyz=0.0925 0.092 -0.160 rpy=0 0 0, axis 1 0 0, limit lower=-0.78 upper=0.78 effort=0.1 velocity=0.1
- added joint right_back_femur_joint: type revolute, parent Right_back_shoulder, child Right_back_femur, origin xyz=0 0.0625 0 rpy=0 0 0, axis 1 0 0, limit lower=-0.78 upper=0.78 effort=0.1 velocity=0.1
- added joint right_back_hip_joint: type revolute, parent base_link, child Right_back_shoulder, origin xyz=-0.0525 0.1125 0.35 rpy=0 0 0, axis 0 1 0, limit lower=-0.78 upper=0.78 effort=0.1 velocity=0.1
- added joint right_back_tibia_joint: type revolute, parent Right_back_femur, child Right_back_tibia, origin xyz=-0.0925 0.092 -0.160 rpy=0 0 0, axis 1 0 0, limit lower=-0.78 upper=0.78 effort=0.1 velocity=0.1
- added joint right_front_femur_joint: type revolute, parent Right_front_shoulder, child Right_front_femur, origin xyz=0.0 -0.0625 0.0 rpy=0 0 0, axis 1 0 0, limit lower=-0.78 upper=0.78 effort=0.1 velocity=0.1
- added joint right_front_hip_joint: type revolute, parent base_link, child Right_front_shoulder, origin xyz=-0.0525 -0.1125 0.35 rpy=0 0 0, axis 0 1 0, limit lower=-0.78 upper=0.78 effort=0.1 velocity=0.1
- added joint right_front_tibia_joint: type revolute, parent Right_front_femur, child Right_front_tibia, origin xyz=-0.0925 0.092 -0.160 rpy=0 0 0, axis 1 0 0, limit lower=-0.78 upper=0.78 effort=0.1 velocity=0.1
