Commit message: Update vrka.xacro

File: vrka_description/urdf/vrka.xacro (robot description, xacro)
@@ -26,5 +26,5 @@
 </link>
 <!--RIGHT FRONT TIBIA -->
-<link name="Right_front_tibia">
+<link name="front_right_lower_leg">
   <inertial>
     <origin rpy="0 0 0" xyz="0.053354897837989246 0.007000373104040586 -0.08200412719516437"/>
@@ -46,8 +46,8 @@
   </collision>
 </link>
-<joint name="Rev30" type="revolute">
+<joint name="motor_front_right_lower_leg" type="revolute">
   <origin rpy="0 0 0" xyz="-0.160214 -0.079 -0.0925"/>
-  <parent link="Right_front_femur"/>
-  <child link="Right_front_tibia"/>
+  <parent link="front_right_upper_leg"/>
+  <child link="front_right_lower_leg"/>
     <limit lower="-0.78" upper="0.78" effort="100" velocity="0.1"/>
   <dynamics damping="0.5"/>
@@ -55,5 +55,5 @@
 </joint>
 <!--RIGHT FRONT FEMUR-->
-<link name="Right_front_femur">
+<link name="front_right_upper_leg">
   <inertial>
     <origin rpy="0 0 0" xyz="-0.02476252170408491 -0.051129281827133444 -0.014293871741900166"/>
@@ -75,8 +75,8 @@
   </collision>
 </link>
-<joint name="Rev31" type="revolute">
+<joint name="motor_front_right_upper_leg" type="revolute">
   <origin rpy="0 0 0" xyz="0.055 -0.0185 0.0"/>
-  <parent link="Right_front_shoulder"/>
-  <child link="Right_front_femur"/>
+  <parent link="front_right_hip"/>
+  <child link="front_right_upper_leg"/>
     <limit lower="-0.78" upper="0.78" effort="100" velocity="0.1"/>
   <dynamics damping="0.5"/>
@@ -84,5 +84,5 @@
 </joint>
 <!--RIGHT FRONT SHOULDER -->
-<link name="Right_front_shoulder">
+<link name="front_right_hip">
   <inertial>
     <origin rpy="0 0 0" xyz="0.055238677027354355 -0.003594806404584705 -2.752506777503605e-07"/>
@@ -104,8 +104,8 @@
   </collision>
 </link>
-<joint name="Rev32" type="revolute">
+<joint name="motor_front_right_hip" type="revolute">
   <origin rpy="0 0 0" xyz="0.140669 -0.094545 0.281084"/>
   <parent link="base_link"/>
-  <child link="Right_front_shoulder"/>
+  <child link="front_right_hip"/>
     <limit lower="-0.78" upper="0.78" effort="100" velocity="0.1"/>
   <dynamics damping="0.5"/>
@@ -113,5 +113,5 @@
 </joint>
 <!--LEFT FRONT TIBIA -->
-<link name="Left_front_tibia">
+<link name="front_left_lower_leg">
   <inertial>
     <origin rpy="0 0 0" xyz="0.05335571926429739 -0.007000189913617491 -0.08200338753311157"/>
@@ -133,8 +133,8 @@
   </collision>
 </link>
-<joint name="Rev33" type="revolute">
+<joint name="motor_front_left_lower_leg" type="revolute">
   <origin rpy="0 0 0" xyz="-0.160215 0.079 -0.0925"/>
-  <parent link="Left_front_femur"/>
-  <child link="Left_front_tibia"/>
+  <parent link="front_left_upper_leg"/>
+  <child link="front_left_lower_leg"/>
     <limit lower="-0.78" upper="0.78" effort="100" velocity="0.1"/>
   <dynamics damping="0.5"/>
@@ -142,5 +142,5 @@
 </joint>
 <!--LEFT FRONT FEMUR -->
-<link name="Left_front_femur">
+<link name="front_left_upper_leg">
   <inertial>
     <origin rpy="0 0 0" xyz="-0.02475988057481357 0.05112942909052748 -0.014298015948625065"/>
@@ -162,8 +162,8 @@
   </collision>
 </link>
-<joint name="Rev34" type="revolute">
+<joint name="motor_front_left_upper_leg" type="revolute">
   <origin rpy="0 0 0" xyz="0.055 0.0185 0.0"/>
-  <parent link="Left_front_shoulder"/>
-  <child link="Left_front_femur"/>
+  <parent link="front_left_hip"/>
+  <child link="front_left_upper_leg"/>
     <limit lower="-0.78" upper="0.78" effort="100" velocity="0.1"/>
   <dynamics damping="0.5"/>
@@ -171,5 +171,5 @@
 </joint>
 <!--LEFT FRONT SHOULDER-->
-<link name="Left_front_shoulder">
+<link name="front_left_hip">
   <inertial>
     <origin rpy="0 0 0" xyz="0.05523849845367643 0.0035949536679779626 3.663911247731022e-07"/>
@@ -191,8 +191,8 @@
   </collision>
 </link>
-<joint name="Rev35" type="revolute">
+<joint name="motor_front_left_hip" type="revolute">
   <origin rpy="0 0 0" xyz="0.140707 0.013252 0.27963"/>
   <parent link="base_link"/>
-  <child link="Left_front_shoulder"/>
+  <child link="front_left_hip"/>
     <limit lower="-0.78" upper="0.78" effort="100" velocity="0.1"/>
   <dynamics damping="0.5"/>
@@ -200,5 +200,5 @@
 </joint>
 <!--RIGHT BACK TIBIA-->
-<link name="Right_back_tibia">
+<link name="back_right_lower_leg">
   <inertial>
     <origin rpy="0 0 0" xyz="0.05335489783801062 0.0070003731040372275 -0.08200412719516668"/>
@@ -220,8 +220,8 @@
   </collision>
 </link>
-<joint name="Rev36" type="revolute">
+<joint name="motor_back_right_lower_leg" type="revolute">
   <origin rpy="0 0 0" xyz="-0.160214 -0.079 -0.0925"/>
-  <parent link="Right_back_femur"/>
-  <child link="Right_back_tibia"/>
+  <parent link="back_right_upper_leg"/>
+  <child link="back_right_lower_leg"/>
   <axis xyz="-0.0 1.0 -0.0"/>
     <limit lower="-0.78" upper="0.78" effort="100" velocity="0.1"/>
@@ -229,5 +229,5 @@
 </joint>
 <!--RIGHT BACK FEMUR -->
-<link name="Right_back_femur">
+<link name="back_right_upper_leg">
   <inertial>
     <origin rpy="0 0 0" xyz="-0.0247625217040503 -0.05112928182713197 -0.014293871741910102"/>
@@ -249,8 +249,8 @@
   </collision>
 </link>
-<joint name="Rev37" type="revolute">
+<joint name="motor_back_right_upper_leg" type="revolute">
   <origin rpy="0 0 0" xyz="-0.055 -0.0185 0.0"/>
-  <parent link="Right_back_shoulder"/>
-  <child link="Right_back_femur"/>
+  <parent link="back_right_hip"/>
+  <child link="back_right_upper_leg"/>
     <limit lower="-0.78" upper="0.78" effort="100" velocity="0.1"/>
   <dynamics damping="0.5"/>
@@ -258,5 +258,5 @@
 </joint>
 <!--RIGHT BACK SHOULDER-->
-<link name="Right_back_shoulder">
+<link name="back_right_hip">
   <inertial>
     <origin rpy="0 0 0" xyz="-0.055238140708366607 -0.0035948064045824013 -3.732709291659475e-07"/>
@@ -278,8 +278,8 @@
   </collision>
 </link>
-<joint name="Rev38" type="revolute">
+<joint name="motor_back_right_hip" type="revolute">
   <origin rpy="0 0 0" xyz="-0.100969 -0.094545 0.281084"/>
   <parent link="base_link"/>
-  <child link="Right_back_shoulder"/>
+  <child link="back_right_hip"/>
     <limit lower="-0.78" upper="0.78" effort="100" velocity="0.1"/>
   <dynamics damping="0.5"/>
@@ -287,5 +287,5 @@
 </joint>
 <!--LEFT BACK TIBIA-->
-<link name="Left_back_tibia">
+<link name="back_left_lower_leg">
   <inertial>
     <origin rpy="0 0 0" xyz="0.053354897838008675 -0.006999626895962993 -0.08200412719516677"/>
@@ -307,8 +307,8 @@
   </collision>
 </link>
-<joint name="Rev39" type="revolute">
+<joint name="motor_back_left_lower_leg" type="revolute">
   <origin rpy="0 0 0" xyz="-0.160214 0.079 -0.0925"/>
-  <parent link="Left_back_femur"/>
-  <child link="Left_back_tibia"/>
+  <parent link="back_left_upper_leg"/>
+  <child link="back_left_lower_leg"/>
   <limit lower="-0.78" upper="0.78" effort="100" velocity="0.1"/>
   <dynamics damping="0.5"/>
@@ -316,5 +316,5 @@
 </joint>
 <!--LEFT BACK FEMUR-->
-<link name="Left_back_femur">
+<link name="back_left_upper_leg">
   <inertial>
     <origin rpy="0 0 0" xyz="-0.024759702001102196 0.05112999210818306 -0.01429875561068078"/>
@@ -336,8 +336,8 @@
   </collision>
 </link>
-<joint name="Rev40" type="revolute">
+<joint name="motor_back_left_upper_leg" type="revolute">
   <origin rpy="0 0 0" xyz="-0.055 0.0185 0.0"/>
-  <parent link="Left_back_shoulder"/>
-  <child link="Left_back_femur"/>
+  <parent link="back_left_hip"/>
+  <child link="back_left_upper_leg"/>
   <limit lower="-0.78" upper="0.78" effort="100" velocity="0.1"/>
   <dynamics damping="0.5"/>
@@ -345,5 +345,5 @@
 </joint>
 <!--LEFT BACK SHOULDER-->
-<link name="Left_back_shoulder">
+<link name="back_left_hip">
   <inertial>
     <origin rpy="0 0 0" xyz="-0.055238140708366884 0.003595516685633909 -2.7525069190570406e-07"/>
@@ -365,8 +365,8 @@
   </collision>
 </link>
-<joint name="Rev41" type="revolute">
+<joint name="motor_back_left_hip" type="revolute">
   <origin rpy="0 0 0" xyz="-0.101049 0.013455 0.281084"/>
   <parent link="base_link"/>
-  <child link="Left_back_shoulder"/>
+  <child link="back_left_hip"/>
   <limit lower="-0.78" upper="0.78" effort="100" velocity="0.1"/>
   <dynamics damping="0.5"/>

Commit message: Update vrka.xacro

File: vrka_description/urdf/vrka.xacro (robot description, xacro)
@@ -54,4 +54,33 @@
   <axis xyz="0.0 1.0 0.0"/>
 </joint>
+<!--right front toe-->
+<link name="front_right_toe">
+  <inertial>
+    <origin rpy="0 -2.1 0 " xyz="0.1 0.009  -0.18"/>
+    <mass value="0.05278821495344609"/>
+    <inertia ixx="4.99e-6" ixy="-0.0" ixz="0.00" iyy="3.99e-6" iyz="0.0" izz="1.99e-6"/>
+  </inertial>
+  <visual>
+    <origin rpy="0 -2.100000 0" xyz="0.11268 -7.955e-3 -0.073584"/>
+    <geometry>
+      <mesh filename="package://vrka_description/meshes/toe_cap1.stl" scale="0.0001 0.0001 0.0001"/>
+    </geometry>
+    <material name="silver"/>
+  </visual>
+  <collision>
+    <origin rpy="0 0 0" xyz="0 0 0"/>
+    <geometry>
+      <mesh filename="package://vrka_description/meshes/toe_cap1.stl" scale="0.0001 0.0001 0.0001"/>
+    </geometry>
+  </collision>
+</link>
+<joint name="motor_front_right_toe" type="revolute">
+  <origin rpy="0 0 0" xyz="0 0 0"/>
+  <parent link="front_right_lower_leg"/>
+  <child link="front_right_toe"/>
+  <axis xyz="-0.0 1.0 -0.0"/>
+    <limit lower="0" upper="0" effort="100" velocity="0.1"/>
+  <dynamics damping="0.5"/>
+</joint>
 <!--RIGHT FRONT FEMUR-->
 <link name="front_right_upper_leg">
@@ -140,4 +169,33 @@
   <dynamics damping="0.5"/>
   <axis xyz="0.0 -1.0 -0.0"/>
+</joint>
+<!--Left front toe-->
+<link name="front_left_toe">
+  <inertial>
+    <origin rpy="0 -2.1 0 " xyz="0.1 -5.3e-3  -0.18"/>
+    <mass value="0.05278821495344609"/>
+    <inertia ixx="4.99e-6" ixy="-0.0" ixz="0.00" iyy="3.99e-6" iyz="0.0" izz="1.99e-6"/>
+  </inertial>
+  <visual>
+    <origin rpy="0 -2.100000 0" xyz="0.11268 -0.02255 -0.073584"/>
+    <geometry>
+      <mesh filename="package://vrka_description/meshes/toe_cap1.stl" scale="0.0001 0.0001 0.0001"/>
+    </geometry>
+    <material name="silver"/>
+  </visual>
+  <collision>
+    <origin rpy="0 0 0" xyz="0 0 0"/>
+    <geometry>
+      <mesh filename="package://vrka_description/meshes/toe_cap1.stl" scale="0.0001 0.0001 0.0001"/>
+    </geometry>
+  </collision>
+</link>
+<joint name="motor_front_left_toe" type="revolute">
+  <origin rpy="0 0 0" xyz="0 0 0"/>
+  <parent link="front_left_lower_leg"/>
+  <child link="front_left_toe"/>
+  <axis xyz="-0.0 1.0 -0.0"/>
+    <limit lower="0" upper="0" effort="100" velocity="0.1"/>
+  <dynamics damping="0.5"/>
 </joint>
 <!--LEFT FRONT FEMUR -->
@@ -228,4 +286,33 @@
   <dynamics damping="0.5"/>
 </joint>
+<!--right back toe test -->
+<link name="back_right_toe">
+  <inertial>
+    <origin rpy="0 -2.1 0 " xyz="0.1 0.009  -0.18"/>
+    <mass value="0.05278821495344609"/>
+    <inertia ixx="4.99e-6" ixy="-0.0" ixz="0.00" iyy="3.99e-6" iyz="0.0" izz="1.99e-6"/>
+  </inertial>
+  <visual>
+    <origin rpy="0 -2.100000 0" xyz="0.113183 -7.955e-3 -0.073584"/>
+    <geometry>
+      <mesh filename="package://vrka_description/meshes/toe_cap1.stl" scale="0.0001 0.0001 0.0001"/>
+    </geometry>
+    <material name="silver"/>
+  </visual>
+  <collision>
+    <origin rpy="0 0 0" xyz="0 0 0"/>
+    <geometry>
+      <mesh filename="package://vrka_description/meshes/toe_cap1.stl" scale="0.0001 0.0001 0.0001"/>
+    </geometry>
+  </collision>
+</link>
+<joint name="motor_back_right_toe" type="revolute">
+  <origin rpy="0 0 0" xyz="0 0 0"/>
+  <parent link="back_right_lower_leg"/>
+  <child link="back_right_toe"/>
+  <axis xyz="-0.0 1.0 -0.0"/>
+    <limit lower="0" upper="0" effort="100" velocity="0.1"/>
+  <dynamics damping="0.5"/>
+</joint>
 <!--RIGHT BACK FEMUR -->
 <link name="back_right_upper_leg">
@@ -315,4 +402,33 @@
   <axis xyz="0.0 -1.0 -0.0"/>
 </joint>
+<!--Left back toe-->
+<link name="back_left_toe">
+  <inertial>
+    <origin rpy="0 -2.1 0 " xyz="0.1 -5.3e-3  -0.18"/>
+    <mass value="0.05278821495344609"/>
+    <inertia ixx="4.99e-6" ixy="-0.0" ixz="0.00" iyy="3.99e-6" iyz="0.0" izz="1.99e-6"/>
+  </inertial>
+  <visual>
+    <origin rpy="0 -2.100000 0" xyz="0.113183 -0.02255 -0.073584"/>
+    <geometry>
+      <mesh filename="package://vrka_description/meshes/toe_cap1.stl" scale="0.0001 0.0001 0.0001"/>
+    </geometry>
+    <material name="silver"/>
+  </visual>
+  <collision>
+    <origin rpy="0 0 0" xyz="0 0 0"/>
+    <geometry>
+      <mesh filename="package://vrka_description/meshes/toe_cap1.stl" scale="0.0001 0.0001 0.0001"/>
+    </geometry>
+  </collision>
+</link>
+<joint name="motor_back_left_toe" type="revolute">
+  <origin rpy="0 0 0" xyz="0 0 0"/>
+  <parent link="back_left_lower_leg"/>
+  <child link="back_left_toe"/>
+  <axis xyz="-0.0 1.0 -0.0"/>
+    <limit lower="0" upper="0" effort="100" velocity="0.1"/>
+  <dynamics damping="0.5"/>
+</joint>
 <!--LEFT BACK FEMUR-->
 <link name="back_left_upper_leg">
